Commit message: changes made to the current setup

File: src/bot/description/warehouse.urdf.xacro (robot description, xacro)
@@ -3,13 +3,62 @@
        xmlns:xacro="http://www.ros.org/wiki/xacro"
        xmlns:ignition="https://ignitionrobotics.org">
-  <xacro:include filename="gazebo_controller.xacro"/>
+  <ros2_control name="IgnitionSystem" type="system">
+    <hardware>
+      <plugin>gz_ros2_control/GazeboSimSystem</plugin>
+    </hardware>
+    <joint name="front_left_wheel_joint">
+      <command_interface name="velocity">
+        <param name="min">-10</param>
+        <param name="max">10</param>
+      </command_interface>
+      <state_interface name="position"/>
+      <state_interface name="velocity"/>
+    </joint>
+    <joint name="front_right_wheel_joint">
+      <command_interface name="velocity">
+        <param name="min">-10</param>
+        <param name="max">10</param>
+      </command_interface>
+      <state_interface name="position"/>
+      <state_interface name="velocity"/>
+    </joint>
+    <joint name="back_left_wheel_joint">
+      <command_interface name="velocity">
+        <param name="min">-10</param>
+        <param name="max">10</param>
+      </command_interface>
+      <state_interface name="position"/>
+      <state_interface name="velocity"/>
+    </joint>
+    <joint name="back_right_wheel_joint">
+      <command_interface name="velocity">
+        <param name="min">-10</param>
+        <param name="max">10</param>
+      </command_interface>
+      <state_interface name="position"/>
+      <state_interface name="velocity"/>
+    </joint>
+  </ros2_control>
+  <gazebo>
+    <plugin filename="libign_ros2_control-system.so"
+            name="ign_ros2_control::IgnitionROS2ControlPlugin">
+      <parameters>$(find bot)/config/controller.yaml</parameters>
+    </plugin>
+  </gazebo>
+  <!-- Base footprint -->
+  <link name="base_footprint"/>
+  <joint name="base_joint" type="fixed">
+    <parent link="base_footprint"/>
+    <child link="base_link"/>
+    <origin xyz="0 0 0" rpy="0 0 0"/>
+  </joint>
   <link name="base_link">
     <inertial>
-      <origin xyz="0.035974 0.020083 6.2148E-05" rpy="0 0 0" />
+      <origin xyz="0.035974 0.020083 6.2148E-05" rpy="0 0 3.14156" />
       <mass value="6.4539" />
       <inertia ixx="0.12648" ixy="-0.0035153" ixz="0.00014021" iyy="0.34337" iyz="-3.3279E-05" izz="0.25605" />
     </inertial>
     <visual>
-      <origin xyz="0 0 0" rpy="0 0 0" />
+      <origin xyz="0 0 0" rpy="0 0 3.14159" />
       <geometry>
         <mesh filename="file://$(find bot)/meshes/base_link.STL" />
@@ -26,4 +75,52 @@
     </collision>
   </link>
+  <!-- Lidar link -->
+  <link name="lidar_link">
+    <visual>
+      <geometry>
+        <cylinder radius="0.05" length="0.05"/>
+      </geometry>
+      <material name=""><color rgba="0.1 0.1 0.1 1" /></material>
+    </visual>
+    <collision>
+      <geometry>
+        <cylinder radius="0.05" length="0.05"/>
+      </geometry>
+    </collision>
+    <inertial>
+      <mass value="0.1"/>
+      <inertia ixx="0.0001" ixy="0" ixz="0" iyy="0.0001" iyz="0" izz="0.0001"/>
+    </inertial>
+  </link>
+  <joint name="lidar_joint" type="fixed">
+    <parent link="base_link"/>
+    <child link="lidar_link"/>
+    <origin xyz="0 0 0.15" rpy="0 0 0"/>
+  </joint>
+  <gazebo reference="lidar_link">
+    <sensor name="lidar" type="gpu_lidar">
+      <always_on>true</always_on>
+      <visualize>true</visualize>
+      <update_rate>10</update_rate>
+      <topic>/scan</topic>
+      <ignition_frame_id>lidar_link</ignition_frame_id>
+      <ray>
+        <scan>
+          <horizontal>
+            <samples>360</samples>
+            <resolution>1.0</resolution>
+            <min_angle>-3.14159</min_angle>
+            <max_angle>3.14159</max_angle>
+          </horizontal>
+        </scan>
+        <range>
+          <min>0.15</min>
+          <max>12.0</max>
+          <resolution>0.01</resolution>
+        </range>
+      </ray>
+    </sensor>
+  </gazebo>
+  <!-- Front Right Wheel -->
   <link name="front_right_wheel">
     <inertial>
@@ -52,4 +149,5 @@
     <axis xyz="0 1 0" />
   </joint>
+  <!-- Front Left Wheel -->
   <link name="front_left_wheel">
     <inertial>
@@ -78,4 +176,5 @@
     <axis xyz="0 1 0" />
   </joint>
+  <!-- Back Left Wheel -->
   <link name="back_left_wheel">
     <inertial>
@@ -104,4 +203,5 @@
     <axis xyz="0 1 0" />
   </joint>
+  <!-- Back Right Wheel -->
   <link name="back_right_wheel">
     <inertial>
@@ -130,4 +230,5 @@
     <axis xyz="0 1 0" />
   </joint>
+  <!-- Wheel friction properties -->
   <gazebo reference="front_left_wheel">
     <collision>
@@ -135,7 +236,7 @@
         <friction>
           <ode>
-            <mu>5.0</mu>
-            <mu2>0.0</mu2>
-            <fdir1 ignition:expressed_in="base_link">1 -1 0</fdir1>
+            <mu>1.0</mu>
+            <mu2>0.2</mu2>
+            <fdir1 ignition:expressed_in="base_footprint">1 -1 0</fdir1>
             <slip1>0.01</slip1>
             <slip2>0.01</slip2>
@@ -144,5 +245,5 @@
         <contact>
           <ode>
-            <kp>1000000.0</kp>
+            <kp>10000000.0</kp>
             <kd>100.0</kd>
             <max_vel>1.0</max_vel>
@@ -158,7 +259,7 @@
         <friction>
           <ode>
-            <mu>5.0</mu>
-            <mu2>0.0</mu2>
-            <fdir1 ignition:expressed_in="base_link">1 1 0</fdir1>
+            <mu>1.0</mu>
+            <mu2>0.2</mu2>
+            <fdir1 ignition:expressed_in="base_footprint">1 1 0</fdir1>
             <slip1>0.01</slip1>
             <slip2>0.01</slip2>
@@ -167,5 +268,5 @@
         <contact>
           <ode>
-            <kp>1000000.0</kp>
+            <kp>10000000.0</kp>
             <kd>100.0</kd>
             <max_vel>1.0</max_vel>
@@ -181,7 +282,7 @@
         <friction>
           <ode>
-            <mu>5.0</mu>
-            <mu2>0.0</mu2>
-            <fdir1 ignition:expressed_in="base_link">1 1 0</fdir1>
+            <mu>1.0</mu>
+            <mu2>0.2</mu2>
+            <fdir1 ignition:expressed_in="base_footprint">1 1 0</fdir1>
             <slip1>0.01</slip1>
             <slip2>0.01</slip2>
@@ -190,5 +291,5 @@
         <contact>
           <ode>
-            <kp>1000000.0</kp>
+            <kp>10000000.0</kp>
             <kd>100.0</kd>
             <max_vel>1.0</max_vel>
@@ -204,7 +305,7 @@
         <friction>
           <ode>
-            <mu>5.0</mu>
-            <mu2>0.0</mu2>
-            <fdir1 ignition:expressed_in="base_link">1 -1 0</fdir1>
+            <mu>1.0</mu>
+            <mu2>0.2</mu2>
+            <fdir1 ignition:expressed_in="base_footprint">1 -1 0</fdir1>
             <slip1>0.01</slip1>
             <slip2>0.01</slip2>
@@ -213,5 +314,5 @@
         <contact>
           <ode>
-            <kp>1000000.0</kp>
+            <kp>10000000.0</kp>
             <kd>100.0</kd>
             <max_vel>1.0</max_vel>
@@ -222,4 +323,5 @@
     </collision>
   </gazebo>
+  <!-- Arm links 1-8 unchanged -->
   <link name="1">
     <inertial>

Commit message: odom issue sorted and all the basic config files added

File: src/bot/description/warehouse.urdf.xacro (robot description, xacro)
@@ -44,4 +44,8 @@
             name="ign_ros2_control::IgnitionROS2ControlPlugin">
       <parameters>$(find bot)/config/controller.yaml</parameters>
+      <ros>
+        <remapping>/mecanum_drive_controller/tf_odometry:=/tf</remapping>
+        <remapping>/mecanum_drive_controller/odometry:=/odom</remapping>
+      </ros>
     </plugin>
   </gazebo>
@@ -122,4 +126,39 @@
     </sensor>
   </gazebo>
+  <!-- IMU SENSOR -->
+  <link name="imu_link">
+    <inertial>
+      <mass value="0.01"/>
+      <origin xyz="0 0 0" rpy="0 0 0"/>
+      <inertia ixx="0.0000166" ixy="0" ixz="0"
+              iyy="0.0000166" iyz="0"
+              izz="0.0000166"/>
+    </inertial>
+  </link>
+  <joint name="imu_joint" type="fixed">
+    <parent link="base_link"/>
+    <child link="imu_link"/>
+    <origin xyz="0 0 0.1" rpy="0 0 0"/>
+  </joint>
+  <gazebo reference="imu_link">
+    <sensor name="imu_sensor" type="imu">
+      <always_on>true</always_on>
+      <update_rate>100</update_rate>
+      <topic>/imu/data</topic>
+      <ignition_frame_id>imu_link</ignition_frame_id>
+      <imu>
+        <angular_velocity>
+          <x><noise type="gaussian"><mean>0</mean><stddev>0.009</stddev></noise></x>
+          <y><noise type="gaussian"><mean>0</mean><stddev>0.009</stddev></noise></y>
+          <z><noise type="gaussian"><mean>0</mean><stddev>0.009</stddev></noise></z>
+        </angular_velocity>
+        <linear_acceleration>
+          <x><noise type="gaussian"><mean>0</mean><stddev>0.021</stddev></noise></x>
+          <y><noise type="gaussian"><mean>0</mean><stddev>0.021</stddev></noise></y>
+          <z><noise type="gaussian"><mean>0</mean><stddev>0.021</stddev></noise></z>
+        </linear_acceleration>
+      </imu>
+    </sensor>
+  </gazebo>
   <!-- Front Right Wheel -->
   <link name="front_right_wheel">
@@ -537,2 +576,3 @@
 <!--fixed the axises-->
 <!--adding the direction of friction and changed the collision geometry to sperical insted of cylindrical-->
+<!--ros2 run teleop_twist_keyboard teleop_twist_keyboard -ros-args -r /cmd_vel:=/mecanum_drive_controller/reference_unstamped-->
